File: Prop_Dev_Stick.sch (EAGLE design)
At the start: 52 parts, among them J1 10118193-0001LF, J3 M20-7822046, J4 M20-7822046, U1 P8X32A-Q44, U2 FT230XQ-R, U4 CAT24C512WI-GT3, U5 AD7999YRJZ-1500RL7, U6 TS2937CW33, U8 TPS2115ADRBR, X1 ATS060CSM-1

Commit message: REV_0B push
Parts:
- L1: device PP_Passives:RESISTOR0603 -> PP_Passives:RESISTOR0402
- U$1: REVNUM REV 2 -> REV 0B
- U4: value CAT24C512WI-GT3 -> CAT24C128WI-GT3
- U6: value TS2937CW33 -> UA78M33CDCYR
Connections:
- net 3.3V: no longer R1.2
- net 5V: now also J3.2, J4.2
- net A0: now also J6.1; no longer J6.2
- net A1: now also J6.3; no longer J6.4
- net GND: now also J6.2, J6.4; no longer J6.1, J6.3
- net IRQ: now also R6.1; no longer R11.1
- net RW: now also R11.1; no longer R6.1
- net SD_CS: now also J3.8, R10.1, U1.P3; no longer J3.5, R7.1, U1.P0
- net SD_DI: now also J3.7, R9.1, U1.P2; no longer J3.6, R8.1, U1.P1
- net SD_DO: now also J3.5, R7.1, U1.P0; no longer J3.8, R10.1, U1.P3
- net SD_SCLK: now also J3.6, R8.1, U1.P1; no longer J3.7, R9.1, U1.P2
- net VBUS_P1: now also R1.2
- net VBUS_P2: no longer J3.2, J4.2
Other:
- moved on the sheet: R10, R11, R6, R7, R8, R9

Commit message: Push Rev 1
Parts:
- L1: device PP_Passives:RESISTOR0402 -> PP_Passives:RESISTOR0603
- U$1: REVNUM REV 0B -> REV 1
- U4: value CAT24C128WI-GT3 -> CAT24C512WI-GT3
- U6: value UA78M33CDCYR -> TS2937CW33
Connections:
- net A0: now also J6.2; no longer J6.1
- net A1: now also J6.4; no longer J6.3
- net GND: now also J6.1, J6.3; no longer J6.2, J6.4
- net IRQ: now also R11.1; no longer R6.1
- net RW: now also R6.1; no longer R11.1
- net SD_CS: now also J3.5, R7.1, U1.P0; no longer J3.8, R10.1, U1.P3
- net SD_DI: now also J3.6, R8.1, U1.P1; no longer J3.7, R9.1, U1.P2
- net SD_DO: now also J3.8, R10.1, U1.P3; no longer J3.5, R7.1, U1.P0
- net SD_SCLK: now also J3.7, R9.1, U1.P2; no longer J3.6, R8.1, U1.P1
Other:
- moved on the sheet: R10, R11, R6, R7, R8, R9
