File: Prop_Dev_Stick.brd (EAGLE design)
At the start: 63.2 x 24.4 mm, 52 parts, among them J1 10118193-0001LF, J3 M20-7822046, J4 M20-7822046, U1 P8X32A-Q44, U2 FT230XQ-R, U4 CAT24C512WI-GT3, U5 AD7999YRJZ-1500RL7, U6 TS2937CW33, U8 TPS2115ADRBR, X1 ATS060CSM-1

Commit message: Fixed Values on a couple parts. Added BOM.txt
Parts:
- J5, J6: value (none) -> M20-7820442
- L1: value MI0603K300R-10 -> MI0603K300R-10
- PWR: value (none) -> 598-8070-107F
- TX/RX: value (none) -> 598-8020-107F
- U7: value (none) -> IRLML6401TRPBF
Changed lines of the file:
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@@
 <attribute name="NAME" x="21.971" y="16.891" size="0.8128" layer="22" font="vector" rot="MR180"/>
 </element>
-<element name="PWR" library="led" package="SML0603" value="" x="2.032" y="18.796" smashed="yes" rot="R180">
+<element name="PWR" library="led" package="SML0603" value="598-8070-107F" x="2.032" y="18.796" smashed="yes" rot="R180">
 <attribute name="NAME" x="5.223" y="20.177" size="0.8128" layer="25" font="vector"/>
 <attribute name="VALUE" x="3.032" y="20.796" size="1.27" layer="27" rot="R180"/>
@@
 <attribute name="NAME" x="3.591" y="19.6215" size="0.8128" layer="25" font="vector"/>
 </element>
-<element name="TX/RX" library="led" package="SML0603" value="" x="7.366" y="7.62" smashed="yes" rot="R180">
+<element name="TX/RX" library="led" package="SML0603" value="598-8020-107F " x="7.366" y="7.62" smashed="yes" rot="R180">
 <attribute name="NAME" x="8.398" y="6.2865" size="0.8128" layer="25" font="vector"/>
 <attribute name="VALUE" x="8.366" y="9.62" size="1.27" layer="27" rot="R180"/>
@@
 <attribute name="NAME" x="50.356" y="17.652" size="0.8128" layer="21" font="vector"/>
 </element>
-<element name="U7" library="PP_DiscreteSemi" package="SOT-23" value="" x="10.287" y="18.288" smashed="yes" rot="R270">
+<element name="U7" library="PP_DiscreteSemi" package="SOT-23" value="IRLML6401TRPBF" x="10.287" y="18.288" smashed="yes" rot="R270">
 <attribute name="NAME" x="11.049" y="15.621" size="0.8128" layer="25" font="vector"/>
 </element>
@@
 <attribute name="NAME" x="7.8105" y="17.942" size="0.8128" layer="25" font="vector" rot="R90"/>
 </element>
-<element name="L1" library="PP_Passives" package="0603" value="  MI0603K300R-10" x="6.096" y="15.621" smashed="yes" rot="R270">
+<element name="L1" library="PP_Passives" package="0603" value="MI0603K300R-10" x="6.096" y="15.621" smashed="yes" rot="R270">
 <attribute name="NAME" x="7.12" y="15.548" size="0.8128" layer="25" font="vector"/>
 </element>
@@
 </element>
 <element name="U$2" library="PP_Aesthetics" package="LHE_LOGO" value="LHE_LOGOLHE_LOGO" x="61.722" y="4.572"/>
-<element name="J5" library="PP_Connectors" package="HEADER_01X04_PTH_ROUND" value="" x="58.42" y="23.622" smashed="yes"/>
-<element name="J6" library="PP_Connectors" package="HEADER_01X04_PTH_ROUND" value="" x="58.42" y="0.762" smashed="yes"/>
+<element name="J5" library="PP_Connectors" package="HEADER_01X04_PTH_ROUND" value="M20-7820442" x="58.42" y="23.622" smashed="yes"/>
+<element name="J6" library="PP_Connectors" package="HEADER_01X04_PTH_ROUND" value="M20-7820442" x="58.42" y="0.762" smashed="yes"/>
 <element name="U5" library="PP_DigitalIC" package="SOT-23-8" value="AD7999YRJZ-1500RL7" x="59.182" y="12.065" smashed="yes">
 <attribute name="NAME" x="55.908" y="9.739" size="0.8128" layer="21" font="vector"/>
@@
 </signal>
 </signals>
-<errors>
-</errors>
 </board>
 </drawing>
